File: connections.kicad_sch (KiCad schematic)
At the start: 17 parts, among them J1 Conn_01x03_Pin, J2 Conn_01x03_Pin, J3 Conn_01x03_Pin, J4 Conn_01x03_Pin, J5 Conn_01x03_Pin, J6 Conn_01x03_Pin

Commit message: cleanup layout, silkmasks, and add connections between planes for power and gnd
Parts:
- J1, J2, J3, J4, J5, J6: now not fitted
Changed lines of the file:
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@@
 		(dnp no)
 		(fields_autoplaced yes)
-		(property "Reference" "#PWR090"
+		(property "Reference" "#PWR0197"
 			(at 58.42 115.57 0)
 			(effects
@@
 			(project ""
 				(path "/d268946a-c85a-4346-a268-ba5c3792dae2/61ec9330-c642-4c33-9122-e615ece33eb7"
-					(reference "#PWR090")
+					(reference "#PWR0197")
 					(unit 1)
 				)
@@
 		(dnp no)
 		(fields_autoplaced yes)
-		(property "Reference" "#PWR022"
+		(property "Reference" "#PWR0202"
 			(at 231.14 153.67 0)
 			(effects
@@
 			(project "ESC BB21"
 				(path "/d268946a-c85a-4346-a268-ba5c3792dae2/61ec9330-c642-4c33-9122-e615ece33eb7"
-					(reference "#PWR022")
+					(reference "#PWR0202")
 					(unit 1)
 				)
@@
 		(on_board yes)
 		(dnp no)
-		(property "Reference" "#PWR019"
+		(property "Reference" "#PWR0199"
 			(at 231.14 129.54 0)
 			(effects
@@
 			(project "ESC BB21"
 				(path "/d268946a-c85a-4346-a268-ba5c3792dae2/61ec9330-c642-4c33-9122-e615ece33eb7"
-					(reference "#PWR019")
+					(reference "#PWR0199")
 					(unit 1)
 				)
@@
 		(dnp no)
 		(fields_autoplaced yes)
-		(property "Reference" "#PWR016"
+		(property "Reference" "#PWR0194"
 			(at 231.14 97.79 0)
 			(effects
@@
 			(project "ESC BB21"
 				(path "/d268946a-c85a-4346-a268-ba5c3792dae2/61ec9330-c642-4c33-9122-e615ece33eb7"
-					(reference "#PWR016")
+					(reference "#PWR0194")
 					(unit 1)
 				)
@@
 		(in_bom yes)
 		(on_board yes)
-		(dnp no)
+		(dnp yes)
 		(property "Reference" "J1"
 			(at 257.81 49.53 0)
@@
 		(dnp no)
 		(fields_autoplaced yes)
-		(property "Reference" "#PWR018"
+		(property "Reference" "#PWR0198"
 			(at 231.14 116.84 0)
 			(effects
@@
 			(project "ESC BB21"
 				(path "/d268946a-c85a-4346-a268-ba5c3792dae2/61ec9330-c642-4c33-9122-e615ece33eb7"
-					(reference "#PWR018")
+					(reference "#PWR0198")
 					(unit 1)
 				)
@@
 		(on_board yes)
 		(dnp no)
-		(property "Reference" "#PWR021"
+		(property "Reference" "#PWR0201"
 			(at 231.14 148.59 0)
 			(effects
@@
 			(project "ESC BB21"
 				(path "/d268946a-c85a-4346-a268-ba5c3792dae2/61ec9330-c642-4c33-9122-e615ece33eb7"
-					(reference "#PWR021")
+					(reference "#PWR0201")
 					(unit 1)
 				)
@@
 		(on_board yes)
 		(dnp no)
-		(property "Reference" "#PWR091"
+		(property "Reference" "#PWR0195"
 			(at 58.42 105.41 0)
 			(effects
@@
 			(project "ESC BB21"
 				(path "/d268946a-c85a-4346-a268-ba5c3792dae2/61ec9330-c642-4c33-9122-e615ece33eb7"
-					(reference "#PWR091")
+					(reference "#PWR0195")
 					(unit 1)
 				)
@@
 		(dnp no)
 		(fields_autoplaced yes)
-		(property "Reference" "#PWR012"
+		(property "Reference" "#PWR0190"
 			(at 231.14 58.42 0)
 			(effects
@@
 			(project "ESC BB21"
 				(path "/d268946a-c85a-4346-a268-ba5c3792dae2/61ec9330-c642-4c33-9122-e615ece33eb7"
-					(reference "#PWR012")
+					(reference "#PWR0190")
 					(unit 1)
 				)
@@
 		(dnp no)
 		(fields_autoplaced yes)
-		(property "Reference" "#PWR014"
+		(property "Reference" "#PWR0192"
 			(at 231.14 77.47 0)
 			(effects
@@
 			(project "ESC BB21"
 				(path "/d268946a-c85a-4346-a268-ba5c3792dae2/61ec9330-c642-4c33-9122-e615ece33eb7"
-					(reference "#PWR014")
+					(reference "#PWR0192")
 					(unit 1)
 				)
@@
 		(in_bom yes)
 		(on_board yes)
-		(dnp no)
+		(dnp yes)
 		(property "Reference" "J2"
 			(at 257.81 68.58 0)
@@
 		(on_board yes)
 		(dnp no)
-		(property "Reference" "#PWR017"
+		(property "Reference" "#PWR0196"
 			(at 231.14 111.76 0)
 			(effects
@@
 			(project "ESC BB21"
 				(path "/d268946a-c85a-4346-a268-ba5c3792dae2/61ec9330-c642-4c33-9122-e615ece33eb7"
-					(reference "#PWR017")
+					(reference "#PWR0196")
 					(unit 1)
 				)
@@
 		(on_board yes)
 		(dnp no)
-		(property "Reference" "#PWR015"
+		(property "Reference" "#PWR0193"
 			(at 231.14 92.71 0)
 			(effects
@@
 			(project "ESC BB21"
 				(path "/d268946a-c85a-4346-a268-ba5c3792dae2/61ec9330-c642-4c33-9122-e615ece33eb7"
-					(reference "#PWR015")
+					(reference "#PWR0193")
 					(unit 1)
 				)
@@
 		(in_bom yes)
 		(on_board yes)
-		(dnp no)
+		(dnp yes)
 		(property "Reference" "J4"
 			(at 257.81 107.95 0)
@@
 		(in_bom yes)
 		(on_board yes)
-		(dnp no)
+		(dnp yes)
 		(property "Reference" "J3"
 			(at 257.81 88.9 0)
@@
 		(on_board yes)
 		(dnp no)
-		(property "Reference" "#PWR013"
+		(property "Reference" "#PWR0191"
 			(at 231.14 72.39 0)
 			(effects
@@
 			(project "ESC BB21"
 				(path "/d268946a-c85a-4346-a268-ba5c3792dae2/61ec9330-c642-4c33-9122-e615ece33eb7"
-					(reference "#PWR013")
+					(reference "#PWR0191")
 					(unit 1)
 				)
@@
 		(on_board yes)
 		(dnp no)
-		(property "Reference" "#PWR011"
+		(property "Reference" "#PWR0189"
 			(at 231.14 53.34 0)
 			(effects
@@
 			(project "ESC BB21"
 				(path "/d268946a-c85a-4346-a268-ba5c3792dae2/61ec9330-c642-4c33-9122-e615ece33eb7"
-					(reference "#PWR011")
+					(reference "#PWR0189")
 					(unit 1)
 				)
@@
 		(in_bom yes)
 		(on_board yes)
-		(dnp no)
+		(dnp yes)
 		(property "Reference" "J6"
 			(at 257.81 144.78 0)
@@
 		(dnp no)
 		(fields_autoplaced yes)
-		(property "Reference" "#PWR020"
+		(property "Reference" "#PWR0200"
 			(at 231.14 134.62 0)
 			(effects
@@
 			(project "ESC BB21"
 				(path "/d268946a-c85a-4346-a268-ba5c3792dae2/61ec9330-c642-4c33-9122-e615ece33eb7"
-					(reference "#PWR020")
+					(reference "#PWR0200")
 					(unit 1)
 				)
@@
 		(in_bom yes)
 		(on_board yes)
-		(dnp no)
+		(dnp yes)
 		(property "Reference" "J5"
 			(at 257.81 125.73 0)
