File: mcu.kicad_sch (KiCad schematic)
At the start: 52 parts, among them SW1 EVPAA602, SW2 EVPAA602, U4 STM32F051K8Tx, U6 STM32F051K8Tx

Commit message: add logo and use 0603 LEDs
Parts:
- D11, D12: footprint ProjectLibrary:LED_0402_1005Metric -> LED_SMD:LED_0603_1608Metric
Changed lines of the file:
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@@
 			)
 		)
-		(property "Footprint" "ProjectLibrary:LED_0402_1005Metric"
+		(property "Footprint" "LED_SMD:LED_0603_1608Metric"
 			(at 139.7 85.09 0)
 			(effects
@@
 			)
 		)
-		(property "Footprint" "ProjectLibrary:LED_0402_1005Metric"
+		(property "Footprint" "LED_SMD:LED_0603_1608Metric"
 			(at 139.7 166.37 0)
 			(effects

Commit message: change LED footprint to 0603 and change D1 to more powerful diode with same footprint
Parts:
- D11, D12: Manufacturer Vishay -> Lite-On; Part Number VLMO1500-GS08 -> LTST-C191KFKT; Voltage (none) -> 2
Changed lines of the file:
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@@
 			)
 		)
-		(property "Manufacturer" "Vishay"
+		(property "Manufacturer" "Lite-On"
 			(at 139.7 85.09 0)
 			(effects
@@
 			)
 		)
-		(property "Part Number" "VLMO1500-GS08 "
+		(property "Part Number" "LTST-C191KFKT"
+			(at 139.7 85.09 0)
+			(effects
+				(font
+					(size 1.27 1.27)
+				)
+				(hide yes)
+			)
+		)
+		(property "Voltage" "2"
 			(at 139.7 85.09 0)
 			(effects
@@
 			)
 		)
-		(property "Manufacturer" "Vishay"
+		(property "Manufacturer" "Lite-On"
+			(at 139.7 166.37 0)
+			(effects
+				(font
+					(size 1.27 1.27)
+				)
+				(hide yes)
+			)
+		)
+		(property "Part Number" "LTST-C191KFKT"
 			(at 139.7 166.37 0)
 			(effects
@@
 			)
 		)
-		(property "Part Number" "VLMO1500-GS08 "
+		(property "Voltage" "2"
 			(at 139.7 166.37 0)
 			(effects

Commit message: remove blind vias
Parts:
- R21, R22, R4, R41, R42, R5: footprint Resistor_SMD:R_0402_1005Metric -> ProjectLibrary:R_0201_0603Metric
- TP10, TP11, TP3, TP4, TP8, TP9: footprint ProjectLibrary:TestPoint_Pad_1.0x1.5mm -> TestPoint:TestPoint_Pad_1.0x1.0mm
- TP5: renamed from TP6; footprint ProjectLibrary:TestPoint_Pad_1.0x1.5mm -> TestPoint:TestPoint_Pad_1.0x1.0mm
- TP6: renamed from TP7; footprint ProjectLibrary:TestPoint_Pad_1.0x1.5mm -> TestPoint:TestPoint_Pad_1.0x1.0mm
- renumbered TP5 to TP7
Connections:
- net +3.3V: now also SW1.1; no longer SW1.2
- net BOOT0_A: now also SW1.2; no longer SW1.1
- net HIN1_A: now also U4.20 (PA10); no longer U4.18 (PA8)
- net HIN1_B: now also U6.20 (PA10); no longer U6.18 (PA8)
- net HIN3_A: now also U4.18 (PA8); no longer U4.20 (PA10)
- net HIN3_B: now also U6.18 (PA8); no longer U6.20 (PA10)
Other:
- note added: "Switched HIN1 and HIN3 for routing"

Commit message: cleanup layout, silkmasks, and add connections between planes for power and gnd
Parts:
- C24: renamed from C22; Tolerance (none) -> 10%
- C25: Tolerance (none) -> 10%
- C26: renamed from C21; Tolerance (none) -> 10%
- C27: renamed from C20; Tolerance (none) -> 10%
- C30: renamed from C33; Tolerance (none) -> 10%
- C31: renamed from C34; Tolerance (none) -> 10%
- C32: renamed from C35; Tolerance (none) -> 10%
- C33: renamed from C36; Tolerance (none) -> 10%
- R10: renamed from R6; Tolerance (none) -> 1%
- R11: renamed from R7; Tolerance (none) -> 1%
- R12: renamed from R8; Tolerance (none) -> 1%
- R13: renamed from R12; Tolerance (none) -> 1%
- R14: renamed from R13; Tolerance (none) -> 1%
- R15: renamed from R14; Tolerance (none) -> 1%
- R16: renamed from R9; Tolerance (none) -> 1%
- R17: renamed from R10; Tolerance (none) -> 1%
- R18: renamed from R11; Tolerance (none) -> 1%
- R20: renamed from R22; Tolerance (none) -> 1%
- R21: renamed from R41; Tolerance (none) -> 1%
- R22: renamed from R23; Tolerance (none) -> 1%
- R23: renamed from R24; Tolerance (none) -> 1%
- R24: renamed from R25; Tolerance (none) -> 1%
- R25: renamed from R26; Tolerance (none) -> 1%
- R26: renamed from R27; Tolerance (none) -> 1%
- R27: renamed from R28; Tolerance (none) -> 1%
- R28: renamed from R29; Tolerance (none) -> 1%
- R29: renamed from R30; Tolerance (none) -> 1%
- R30: renamed from R31; Tolerance (none) -> 1%
- R8: renamed from R4; Tolerance (none) -> 1%
- R9: renamed from R42; Tolerance (none) -> 1%
- renumbered C26 to C28, C27 to C29, C37 to C34, C38 to C35, D12 to D5, D11 to D6, R21 to R19, R5 to R7, U4 to U5
Other:
- note added: "Voltage dividers from 5 to 3.3V"

Commit message: cleanup BOM and bump up voltage rating/footprint for capacitors to max possible
Parts:
- C24, C29, C30, C35: footprint Capacitor_SMD:C_0402_1005Metric -> Capacitor_SMD:C_0603_1608Metric; Manufacturer YAGEO -> Murata; Part Number GRM155R61E102KA01D -> GRM188R61E106KA73D; Voltage 10 -> 25
- C25, C26, C27, C28, C31, C32, C33, C34: Manufacturer YAGEO -> Murata; Part Number CC0402KRX5R7BB104 -> GRM155R61H104KE14D; Voltage 16 -> 50
Changed lines of the file:
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@@
 			)
 		)
-		(property "Part Number" "CC0402KRX5R7BB104"
+		(property "Part Number" "GRM155R61H104KE14D"
 			(at 92.71 111.76 0)
 			(effects
@@
 			)
 		)
-		(property "Manufacturer" "YAGEO"
+		(property "Manufacturer" "Murata"
 			(at 92.71 111.76 0)
 			(effects
@@
 			)
 		)
-		(property "Voltage" "16"
+		(property "Voltage" "50"
 			(at 92.71 111.76 0)
 			(effects
@@
 			)
 		)
-		(property "Part Number" "CC0402KRX5R7BB104"
+		(property "Part Number" "GRM155R61H104KE14D"
 			(at 85.09 30.48 0)
 			(effects
@@
 			)
 		)
-		(property "Manufacturer" "YAGEO"
+		(property "Manufacturer" "Murata"
 			(at 85.09 30.48 0)
 			(effects
@@
 			)
 		)
-		(property "Voltage" "16"
+		(property "Voltage" "50"
 			(at 85.09 30.48 0)
 			(effects
@@
 			)
 		)
-		(property "Part Number" "CC0402KRX5R7BB104"
+		(property "Part Number" "GRM155R61H104KE14D"
 			(at 77.47 43.18 0)
 			(effects
@@
 			)
 		)
-		(property "Manufacturer" "YAGEO"
+		(property "Manufacturer" "Murata"
 			(at 77.47 43.18 0)
 			(effects
@@
 			)
 		)
-		(property "Voltage" "16"
+		(property "Voltage" "50"
 			(at 77.47 43.18 0)
 			(effects
@@
 			)
 		)
-		(property "Footprint" "Capacitor_SMD:C_0402_1005Metric"
+		(property "Footprint" "Capacitor_SMD:C_0603_1608Metric"
 			(at 122.8852 115.57 0)
 			(effects
@@
 			)
 		)
-		(property "Part Number" "GRM155R61E102KA01D"
+		(property "Part Number" "GRM188R61E106KA73D"
 			(at 121.92 111.76 0)
 			(effects
@@
 			)
 		)
-		(property "Voltage" "10"
+		(property "Voltage" "25"
 			(at 121.92 111.76 0)
 			(effects
@@
 			)
 		)
-		(property "Manufacturer" "YAGEO"
+		(property "Manufacturer" "Murata"
 			(at 121.92 111.76 0)
 			(effects
@@
 			)
 		)
-		(property "Footprint" "Capacitor_SMD:C_0402_1005Metric"
+		(property "Footprint" "Capacitor_SMD:C_0603_1608Metric"
 			(at 122.8852 34.29 0)
 			(effects
@@
 			)
 		)
-		(property "Part Number" "GRM155R61E102KA01D"
+		(property "Part Number" "GRM188R61E106KA73D"
 			(at 121.92 30.48 0)
 			(effects
@@
 			)
 		)
-		(property "Voltage" "10"
+		(property "Voltage" "25"
 			(at 121.92 30.48 0)
 			(effects
@@
 			)
 		)
-		(property "Manufacturer" "YAGEO"
+		(property "Manufacturer" "Murata"
 			(at 121.92 30.48 0)
 			(effects
@@
 			)
 		)
-		(property "Datasheet" "EVP-AA602W"
+		(property "Datasheet" "https://www3.panasonic.biz/ac/cdn/e/control/switch/light-touch/catalog/sw_lt_eng_3529s.pdf"
 			(at 46.99 45.72 0)
 			(effects
@@
 			)
 		)
-		(property "Part Number" "CC0402KRX5R7BB104"
+		(property "Part Number" "GRM155R61H104KE14D"
 			(at 114.3 30.48 0)
 			(effects
@@
 			)
 		)
-		(property "Voltage" "16"
+		(property "Voltage" "50"
 			(at 114.3 30.48 0)
 			(effects
@@
 			)
 		)
-		(property "Manufacturer" "YAGEO"
+		(property "Manufacturer" "Murata"
 			(at 114.3 30.48 0)
 			(effects
@@
 			)
 		)
-		(property "Part Number" "CC0402KRX5R7BB104"
+		(property "Part Number" "GRM155R61H104KE14D"
 			(at 85.09 111.76 0)
 			(effects
@@
 			)
 		)
-		(property "Manufacturer" "YAGEO"
+		(property "Manufacturer" "Murata"
 			(at 85.09 111.76 0)
 			(effects
@@
 			)
 		)
-		(property "Voltage" "16"
+		(property "Voltage" "50"
 			(at 85.09 111.76 0)
 			(effects
@@
 			)
 		)
-		(property "Part Number" "CC0402KRX5R7BB104"
+		(property "Part Number" "GRM155R61H104KE14D"
 			(at 114.3 111.76 0)
 			(effects
@@
 			)
 		)
-		(property "Voltage" "16"
+		(property "Voltage" "50"
 			(at 114.3 111.76 0)
 			(effects
@@
 			)
 		)
-		(property "Manufacturer" "YAGEO"
+		(property "Manufacturer" "Murata"
 			(at 114.3 111.76 0)
 			(effects
@@
 			)
 		)
-		(property "Datasheet" "EVP-AA602W"
+		(property "Datasheet" "https://www3.panasonic.biz/ac/cdn/e/control/switch/light-touch/catalog/sw_lt_eng_3529s.pdf"
 			(at 46.99 127 0)
 			(effects
@@
 			)
 		)
-		(property "Footprint" "Capacitor_SMD:C_0402_1005Metric"
+		(property "Footprint" "Capacitor_SMD:C_0603_1608Metric"
 			(at 78.4352 34.29 0)
 			(effects
@@
 			)
 		)
-		(property "Part Number" "GRM155R61E102KA01D"
+		(property "Part Number" "GRM188R61E106KA73D"
 			(at 77.47 30.48 0)
 			(effects
@@
 			)
 		)
-		(property "Manufacturer" "YAGEO"
+		(property "Manufacturer" "Murata"
 			(at 77.47 30.48 0)
 			(effects
@@
 			)
 		)
-		(property "Voltage" "10"
+		(property "Voltage" "25"
 			(at 77.47 30.48 0)
 			(effects
@@
 			)
 		)
-		(property "Footprint" "Capacitor_SMD:C_0402_1005Metric"
+		(property "Footprint" "Capacitor_SMD:C_0603_1608Metric"
 			(at 78.4352 115.57 0)
 			(effects
@@
 			)
 		)
-		(property "Part Number" "GRM155R61E102KA01D"
+		(property "Part Number" "GRM188R61E106KA73D"
 			(at 77.47 111.76 0)
 			(effects
@@
 			)
 		)
-		(property "Manufacturer" "YAGEO"
+		(property "Manufacturer" "Murata"
 			(at 77.47 111.76 0)
 			(effects
@@
 			)
 		)
-		(property "Voltage" "10"
+		(property "Voltage" "25"
 			(at 77.47 111.76 0)
 			(effects
@@
 			)
 		)
-		(property "Part Number" "CC0402KRX5R7BB104"
+		(property "Part Number" "GRM155R61H104KE14D"
 			(at 92.71 30.48 0)
 			(effects
@@
 			)
 		)
-		(property "Manufacturer" "YAGEO"
+		(property "Manufacturer" "Murata"
 			(at 92.71 30.48 0)
 			(effects
@@
 			)
 		)
-		(property "Voltage" "16"
+		(property "Voltage" "50"
 			(at 92.71 30.48 0)
 			(effects
@@
 			)
 		)
-		(property "Part Number" "CC0402KRX5R7BB104"
+		(property "Part Number" "GRM155R61H104KE14D"
 			(at 77.47 124.46 0)
 			(effects
@@
 			)
 		)
-		(property "Manufacturer" "YAGEO"
+		(property "Manufacturer" "Murata"
 			(at 77.47 124.46 0)
 			(effects
@@
 			)
 		)
-		(property "Voltage" "16"
+		(property "Voltage" "50"
 			(at 77.47 124.46 0)
 			(effects
