File: power.kicad_sch (KiCad schematic)
At the start: 43 parts, among them U1 INA190A4IDCKR, U2 MAX20008AFOA/VY+, U3 AP63205WU, U4 AP63203WU

Commit message: cleanup BOM and bump up voltage rating/footprint for capacitors to max possible
Parts:
- C13: Part Number GRM155R61E102KA01D -> GRM155R61H102KA01D; Voltage (none) -> 50
- C15, C19, C5, C6: Manufacturer YAGEO -> Murata; Part Number CC0402KRX5R7BB104 -> GRM155R61H104KE14D; Voltage 16 -> 50
- C2: Manufacturer YAGEO -> Murata; Part Number CC0402KRX5R7BB225 -> GRM155R6YA225KE11D; Voltage 16 -> 35
Changed lines of the file:
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@@
 			)
 		)
-		(property "Manufacturer" "YAGEO"
+		(property "Manufacturer" "Murata"
 			(at 80.01 96.52 0)
 			(effects
@@
 			)
 		)
-		(property "Part Number" "CC0402KRX5R7BB225 "
+		(property "Part Number" "GRM155R6YA225KE11D"
 			(at 80.01 96.52 0)
 			(effects
@@
 			)
 		)
-		(property "Voltage" "16"
+		(property "Voltage" "35"
 			(at 80.01 96.52 0)
 			(effects
@@
 			)
 		)
-		(property "Manufacturer" "YAGEO"
+		(property "Manufacturer" "Murata"
 			(at 100.33 110.49 0)
 			(effects
@@
 			)
 		)
-		(property "Part Number" "CC0402KRX5R7BB104"
+		(property "Part Number" "GRM155R61H104KE14D"
 			(at 100.33 110.49 0)
 			(effects
@@
 			)
 		)
-		(property "Voltage" "16"
+		(property "Voltage" "50"
 			(at 100.33 110.49 0)
 			(effects
@@
 			)
 		)
-		(property "Datasheet" "~"
+		(property "Datasheet" "https://www.bourns.com/docs/product-datasheets/1-5smbj.pdf"
 			(at 62.23 29.21 0)
 			(effects
@@
 			)
 		)
-		(property "Part Number" "CC0402KRX5R7BB104"
+		(property "Part Number" "GRM155R61H104KE14D"
 			(at 88.9 139.7 0)
 			(effects
@@
 			)
 		)
-		(property "Voltage" "16"
+		(property "Voltage" "50"
 			(at 88.9 139.7 0)
 			(effects
@@
 			)
 		)
-		(property "Manufacturer" "YAGEO"
+		(property "Manufacturer" "Murata"
 			(at 88.9 139.7 0)
 			(effects
@@
 			)
 		)
-		(property "Part Number" "CC0402KRX5R7BB104"
+		(property "Part Number" "GRM155R61H104KE14D"
 			(at 189.23 140.97 0)
 			(effects
@@
 			)
 		)
-		(property "Voltage" "16"
+		(property "Voltage" "50"
 			(at 189.23 140.97 0)
 			(effects
@@
 			)
 		)
-		(property "Manufacturer" "YAGEO"
+		(property "Manufacturer" "Murata"
 			(at 189.23 140.97 0)
 			(effects
@@
 			)
 		)
-		(property "Datasheet" "INA190A4IDCKR"
+		(property "Datasheet" "https://www.ti.com/general/docs/suppproductinfo.tsp?distId=10&gotoUrl=https%3A%2F%2Fwww.ti.com%2Flit%2Fgpn%2Fina190"
 			(at 101.6 35.56 0)
 			(effects
@@
 			)
 		)
-		(property "Manufacturer" "YAGEO"
+		(property "Manufacturer" "Murata"
 			(at 161.29 95.25 0)
 			(effects
@@
 			)
 		)
-		(property "Part Number" "CC0402KRX5R7BB104"
+		(property "Part Number" "GRM155R61H104KE14D"
 			(at 161.29 95.25 0)
 			(effects
@@
 			)
 		)
-		(property "Voltage" "16"
+		(property "Voltage" "50"
 			(at 161.29 95.25 0)
 			(effects
@@
 			)
 		)
-		(property "Part Number" "GRM155R61E102KA01D"
+		(property "Part Number" "GRM155R61H102KA01D"
 			(at 231.14 97.79 0)
 			(effects
@@
 			)
 		)
+		(property "Voltage" "50"
+			(at 231.14 97.79 0)
+			(effects
+				(font
+					(size 1.27 1.27)
+				)
+				(hide yes)
+			)
+		)
 		(pin "2"
 		)
@@
 			)
 		)
-		(property "Datasheet" "MAX20008AFOC/VY+T"
+		(property "Datasheet" "https://www.analog.com/media/en/technical-documentation/data-sheets/MAX20004-MAX20008.pdf"
 			(at 146.05 86.36 0)
 			(effects
